Commit message: ROS added

File: robot_sim/description/robot.urdf.xacro (robot description, xacro)
@@ -8,6 +8,6 @@
     <inertial><mass value="5"/><inertia ixx="0.1" ixy="0" ixz="0" iyy="0.1" iyz="0" izz="0.1"/></inertial>
   </link>
-  <link name="left_wheel"><visual><geometry><cylinder radius="0.1" length="0.06"/></geometry><material name="black"/></visual><collision><geometry><cylinder radius="0.1" length="0.06"/></geometry></collision></link>
-  <link name="right_wheel"><visual><geometry><cylinder radius="0.1" length="0.06"/></geometry><material name="black"/></visual><collision><geometry><cylinder radius="0.1" length="0.06"/></geometry></collision></link>
+  <link name="left_wheel"><visual><geometry><cylinder radius="0.1" length="0.06"/></geometry><material name="black"/></visual><collision><geometry><cylinder radius="0.1" length="0.06"/></geometry></collision><inertial><mass value="0.5"/><inertia ixx="0.0014" ixy="0" ixz="0" iyy="0.0014" iyz="0" izz="0.0025"/></inertial></link>
+  <link name="right_wheel"><visual><geometry><cylinder radius="0.1" length="0.06"/></geometry><material name="black"/></visual><collision><geometry><cylinder radius="0.1" length="0.06"/></geometry></collision><inertial><mass value="0.5"/><inertia ixx="0.0014" ixy="0" ixz="0" iyy="0.0014" iyz="0" izz="0.0025"/></inertial></link>
   <joint name="left_wheel_joint" type="continuous">
     <parent link="base_link"/><child link="left_wheel"/><origin xyz="0 0.23 -0.03" rpy="1.5708 0 0"/><axis xyz="0 0 1"/>
@@ -16,4 +16,13 @@
     <parent link="base_link"/><child link="right_wheel"/><origin xyz="0 -0.23 -0.03" rpy="1.5708 0 0"/><axis xyz="0 0 1"/>
   </joint>
+  <link name="caster">
+    <visual><geometry><sphere radius="0.05"/></geometry><material name="black"/></visual>
+    <collision><geometry><sphere radius="0.05"/></geometry></collision>
+    <inertial><mass value="0.1"/><inertia ixx="0.0001" ixy="0" ixz="0" iyy="0.0001" iyz="0" izz="0.0001"/></inertial>
+  </link>
+  <joint name="caster_joint" type="fixed">
+    <parent link="base_link"/><child link="caster"/><origin xyz="-0.22 0 -0.08"/>
+  </joint>
+  <gazebo reference="caster"><mu1>0</mu1><mu2>0</mu2></gazebo>
   <gazebo reference="base_link"><material>Gazebo/Blue</material></gazebo>
   <gazebo>
@@ -28,4 +37,7 @@
       <child_frame_id>base_link</child_frame_id>
     </plugin>
+    <plugin filename="gz-sim-joint-state-publisher-system" name="gz::sim::systems::JointStatePublisher">
+      <topic>/joint_states</topic>
+    </plugin>
   </gazebo>
 </robot>

Commit message: fixed the readme

File: robot_sim/description/robot.urdf.xacro (robot description, xacro)
@@ -1,33 +1,69 @@
 <?xml version="1.0"?>
 <robot name="robot" xmlns:xacro="http://www.ros.org/wiki/xacro">
-  <material name="blue"><color rgba="0.05 0.25 0.8 1"/></material>
+  <xacro:property name="length" value="0.9"/>
+  <xacro:property name="width"  value="0.4"/>
+  <xacro:property name="height" value="0.18"/>
+  <xacro:property name="mass"   value="5"/>
+  <xacro:property name="wheel_x" value="0.3"/>
+  <xacro:property name="wheel_y" value="0.23"/>
+  <material name="red"><color rgba="0.8 0.05 0.05 1"/></material>
   <material name="black"><color rgba="0.03 0.03 0.03 1"/></material>
   <link name="base_link">
-    <visual><geometry><box size="0.6 0.4 0.18"/></geometry><material name="blue"/></visual>
-    <collision><geometry><box size="0.6 0.4 0.18"/></geometry></collision>
-    <inertial><mass value="5"/><inertia ixx="0.1" ixy="0" ixz="0" iyy="0.1" iyz="0" izz="0.1"/></inertial>
+    <visual><geometry><box size="${length} ${width} ${height}"/></geometry><material name="red"/></visual>
+    <collision><geometry><box size="${length} ${width} ${height}"/></geometry></collision>
+    <inertial>
+      <mass value="${mass}"/>
+      <inertia ixx="${mass*(width*width+height*height)/12}" ixy="0" ixz="0"
+               iyy="${mass*(length*length+height*height)/12}" iyz="0"
+               izz="${mass*(length*length+width*width)/12}"/>
+    </inertial>
   </link>
-  <link name="left_wheel"><visual><geometry><cylinder radius="0.1" length="0.06"/></geometry><material name="black"/></visual><collision><geometry><cylinder radius="0.1" length="0.06"/></geometry></collision><inertial><mass value="0.5"/><inertia ixx="0.0014" ixy="0" ixz="0" iyy="0.0014" iyz="0" izz="0.0025"/></inertial></link>
-  <link name="right_wheel"><visual><geometry><cylinder radius="0.1" length="0.06"/></geometry><material name="black"/></visual><collision><geometry><cylinder radius="0.1" length="0.06"/></geometry></collision><inertial><mass value="0.5"/><inertia ixx="0.0014" ixy="0" ixz="0" iyy="0.0014" iyz="0" izz="0.0025"/></inertial></link>
-  <joint name="left_wheel_joint" type="continuous">
-    <parent link="base_link"/><child link="left_wheel"/><origin xyz="0 0.23 -0.03" rpy="1.5708 0 0"/><axis xyz="0 0 1"/>
+  <xacro:macro name="wheel" params="name x y">
+    <link name="${name}">
+      <visual><geometry><cylinder radius="0.1" length="0.06"/></geometry><material name="black"/></visual>
+      <collision><geometry><cylinder radius="0.1" length="0.06"/></geometry></collision>
+      <inertial><mass value="0.5"/><inertia ixx="0.0014" ixy="0" ixz="0" iyy="0.0014" iyz="0" izz="0.0025"/></inertial>
+    </link>
+    <joint name="${name}_joint" type="continuous">
+      <parent link="base_link"/><child link="${name}"/>
+      <origin xyz="${x} ${y} -0.03" rpy="-1.5708 0 0"/><axis xyz="0 0 1"/>
+    </joint>
+    <gazebo reference="${name}"><mu1>1.0</mu1><mu2>0.1</mu2></gazebo>
+  </xacro:macro>
+  <xacro:wheel name="front_left_wheel"  x="${wheel_x}"  y="${wheel_y}"/>
+  <xacro:wheel name="front_right_wheel" x="${wheel_x}"  y="${-wheel_y}"/>
+  <xacro:wheel name="rear_left_wheel"   x="${-wheel_x}" y="${wheel_y}"/>
+  <xacro:wheel name="rear_right_wheel"  x="${-wheel_x}" y="${-wheel_y}"/>
+<!-- FLAG REMOVE THIS MR.TAMIM ONCE DONE ALRIGHT -->
+  <material name="white"><color rgba="0.95 0.95 0.95 1"/></material>
+  <material name="yellow"><color rgba="1 0.85 0.1 1"/></material>
+  <link name="flag_pole">
+    <visual><geometry><cylinder radius="0.01" length="0.5"/></geometry><material name="white"/></visual>
+    <collision><geometry><cylinder radius="0.01" length="0.5"/></geometry></collision>
+    <inertial><mass value="0.05"/><inertia ixx="0.0001" ixy="0" ixz="0" iyy="0.0001" iyz="0" izz="0.0001"/></inertial>
+  </link>
+  <joint name="flag_pole_joint" type="fixed">
+    <parent link="base_link"/><child link="flag_pole"/>
+    <origin xyz="${-length/2 + 0.05} 0 ${height/2 + 0.25}"/>
   </joint>
-  <joint name="right_wheel_joint" type="continuous">
-    <parent link="base_link"/><child link="right_wheel"/><origin xyz="0 -0.23 -0.03" rpy="1.5708 0 0"/><axis xyz="0 0 1"/>
+  <link name="flag">
+    <visual>
+      <geometry><box size="0.8 0.01 0.2"/></geometry>
+      <material name="yellow"/>
+    </visual>
+    <collision><geometry><box size="0.8 0.01 0.2"/></geometry></collision>
+    <inertial><mass value="0.05"/><inertia ixx="0.0001" ixy="0" ixz="0" iyy="0.0001" iyz="0" izz="0.0001"/></inertial>
+  </link>
+  <joint name="flag_joint" type="fixed">
+    <parent link="flag_pole"/><child link="flag"/>
+    <origin xyz="-0.4 0 0.15"/>
   </joint>
-  <link name="caster">
-    <visual><geometry><sphere radius="0.05"/></geometry><material name="black"/></visual>
-    <collision><geometry><sphere radius="0.05"/></geometry></collision>
-    <inertial><mass value="0.1"/><inertia ixx="0.0001" ixy="0" ixz="0" iyy="0.0001" iyz="0" izz="0.0001"/></inertial>
-  </link>
-  <joint name="caster_joint" type="fixed">
-    <parent link="base_link"/><child link="caster"/><origin xyz="-0.22 0 -0.08"/>
-  </joint>
-  <gazebo reference="caster"><mu1>0</mu1><mu2>0</mu2></gazebo>
-  <gazebo reference="base_link"><material>Gazebo/Blue</material></gazebo>
+<!-- HERE IS THE END OF GLAG -->
   <gazebo>
     <plugin filename="gz-sim-diff-drive-system" name="gz::sim::systems::DiffDrive">
-      <left_joint>left_wheel_joint</left_joint>
-      <right_joint>right_wheel_joint</right_joint>
+      <left_joint>front_left_wheel_joint</left_joint>
+      <left_joint>rear_left_wheel_joint</left_joint>
+      <right_joint>front_right_wheel_joint</right_joint>
+      <right_joint>rear_right_wheel_joint</right_joint>
       <wheel_separation>0.46</wheel_separation>
       <wheel_radius>0.1</wheel_radius>

Commit message: fixed flag

File: robot_sim/description/robot.urdf.xacro (robot description, xacro)
@@ -49,13 +49,13 @@
   <link name="flag">
     <visual>
-      <geometry><box size="0.8 0.01 0.2"/></geometry>
+      <geometry><box size="0.5 0.01 0.2"/></geometry>
       <material name="yellow"/>
     </visual>
-    <collision><geometry><box size="0.8 0.01 0.2"/></geometry></collision>
+    <collision><geometry><box size="0.5 0.01 0.2"/></geometry></collision>
     <inertial><mass value="0.05"/><inertia ixx="0.0001" ixy="0" ixz="0" iyy="0.0001" iyz="0" izz="0.0001"/></inertial>
   </link>
   <joint name="flag_joint" type="fixed">
     <parent link="flag_pole"/><child link="flag"/>
-    <origin xyz="-0.4 0 0.15"/>
+    <origin xyz="-0.25 0 0.15"/>
   </joint>
 <!-- HERE IS THE END OF GLAG -->
